File: rosekicad/rosekicad.kicad_pcb (KiCad board)
At the start: 2 copper layers, 26 parts, among them Q1 2N2222, Q10 2N2222, Q11 2N2222, Q12 2N2222, Q13 2N2222, Q14 2N2222, Q15 2N2222, Q2 2N2222, Q3 2N2222, Q4 2N2222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

Commit message: updated footprints
Parts:
- added C1: 470 uF, Capacitor_THT:CP_Radial_D10.0mm_P3.80mm, F.Cu at (133.2, 29.4)
- added C2: 470 uF, Capacitor_THT:CP_Radial_D10.0mm_P3.80mm, F.Cu at (133.2, 41.0)
- added C3: 470 uF, Capacitor_THT:CP_Radial_D10.0mm_P3.80mm, F.Cu at (133.2, 52.5)
- added C4: 0.1u, Capacitor_THT:CP_Radial_D5.0mm_P2.00mm, F.Cu at (175.5, 57.2)
- added C5: 470 uF, Capacitor_THT:CP_Radial_D10.0mm_P3.80mm, F.Cu at (133.2, 64.1)
- added J1: Solenoid, TerminalBlock:TerminalBlock_MaiXu_MX126-5.0-02P_1x02_P5.00mm, F.Cu at (177.2, 28.7)
- added J10: Solenoid, TerminalBlock:TerminalBlock_MaiXu_MX126-5.0-02P_1x02_P5.00mm, F.Cu at (162.4, 99.5)
- added J11: Solenoid, TerminalBlock:TerminalBlock_MaiXu_MX126-5.0-02P_1x02_P5.00mm, F.Cu at (180.0, 69.2)
- added J12: Solenoid, TerminalBlock:TerminalBlock_MaiXu_MX126-5.0-02P_1x02_P5.00mm, F.Cu at (180.0, 79.3)
- added J13: UV Lights, TerminalBlock:TerminalBlock_MaiXu_MX126-5.0-02P_1x02_P5.00mm, F.Cu at (180.0, 89.4)
- added J14: LED Lights, TerminalBlock:TerminalBlock_MaiXu_MX126-5.0-02P_1x02_P5.00mm, F.Cu at (180.0, 99.5)
- added J15: DMX Cable, TerminalBlock:TerminalBlock_MaiXu_MX126-5.0-05P_1x05_P5.00mm, F.Cu at (177.2, 48.9)
- added J16: Barrel_Jack_MountingPin, Connector_BarrelJack:BarrelJack_CUI_PJ-102AH_Horizontal, F.Cu at (228.8, 30.3)
- added J2: Solenoid, TerminalBlock:TerminalBlock_MaiXu_MX126-5.0-02P_1x02_P5.00mm, F.Cu at (177.2, 38.8)
- added J3: Solenoid, TerminalBlock:TerminalBlock_MaiXu_MX126-5.0-02P_1x02_P5.00mm, F.Cu at (144.9, 69.2)
- added J4: Solenoid, TerminalBlock:TerminalBlock_MaiXu_MX126-5.0-02P_1x02_P5.00mm, F.Cu at (144.9, 79.3)
- added J5: Solenoid, TerminalBlock:TerminalBlock_MaiXu_MX126-5.0-02P_1x02_P5.00mm, F.Cu at (144.9, 89.4)
- added J6: Solenoid, TerminalBlock:TerminalBlock_MaiXu_MX126-5.0-02P_1x02_P5.00mm, F.Cu at (144.9, 99.5)
- added J7: Solenoid, TerminalBlock:TerminalBlock_MaiXu_MX126-5.0-02P_1x02_P5.00mm, F.Cu at (162.4, 69.2)
- added J8: Solenoid, TerminalBlock:TerminalBlock_MaiXu_MX126-5.0-02P_1x02_P5.00mm, F.Cu at (162.4, 79.3)
- added J9: Solenoid, TerminalBlock:TerminalBlock_MaiXu_MX126-5.0-02P_1x02_P5.00mm, F.Cu at (162.4, 89.4)
- added R1: 220, Resistor_THT:R_Axial_DIN0207_L6.3mm_D2.5mm_P7.62mm_Horizontal, F.Cu at (142.4, 25.7)
- added R10: 220, Resistor_THT:R_Axial_DIN0207_L6.3mm_D2.5mm_P7.62mm_Horizontal, F.Cu at (142.4, 62.1)
- added R11: 2.2, Resistor_THT:R_Axial_DIN0207_L6.3mm_D2.5mm_P7.62mm_Horizontal, F.Cu at (153.2, 25.7)
- added R12: 2.2, Resistor_THT:R_Axial_DIN0207_L6.3mm_D2.5mm_P7.62mm_Horizontal, F.Cu at (153.2, 29.7)
- added R13: 2.2, Resistor_THT:R_Axial_DIN0207_L6.3mm_D2.5mm_P7.62mm_Horizontal, F.Cu at (153.2, 33.8)
- added R14: 2.2, Resistor_THT:R_Axial_DIN0207_L6.3mm_D2.5mm_P7.62mm_Horizontal, F.Cu at (153.2, 37.8)
- added R15: 100, Resistor_THT:R_Axial_DIN0207_L6.3mm_D2.5mm_P7.62mm_Horizontal, F.Cu at (153.2, 41.9)
- added R16: 100, Resistor_THT:R_Axial_DIN0207_L6.3mm_D2.5mm_P7.62mm_Horizontal, F.Cu at (153.2, 45.9)
- added R17: 100, Resistor_THT:R_Axial_DIN0207_L6.3mm_D2.5mm_P7.62mm_Horizontal, F.Cu at (153.2, 50.0)
- added R18: 100, Resistor_THT:R_Axial_DIN0207_L6.3mm_D2.5mm_P7.62mm_Horizontal, F.Cu at (153.2, 54.0)
- added R19: 220, Resistor_THT:R_Axial_DIN0207_L6.3mm_D2.5mm_P7.62mm_Horizontal, F.Cu at (153.2, 58.1)
- added R2: 2.2, Resistor_THT:R_Axial_DIN0207_L6.3mm_D2.5mm_P7.62mm_Horizontal, F.Cu at (142.4, 29.7)
- added R20: 2.2, Resistor_THT:R_Axial_DIN0207_L6.3mm_D2.5mm_P7.62mm_Horizontal, F.Cu at (153.2, 62.1)
- added R21: 2.2, Resistor_THT:R_Axial_DIN0207_L6.3mm_D2.5mm_P7.62mm_Horizontal, F.Cu at (164.0, 25.7)
- added R22: 2.2, Resistor_THT:R_Axial_DIN0207_L6.3mm_D2.5mm_P7.62mm_Horizontal, F.Cu at (164.0, 29.7)
- added R23: 2.2, Resistor_THT:R_Axial_DIN0207_L6.3mm_D2.5mm_P7.62mm_Horizontal, F.Cu at (164.0, 33.8)
- added R24: 100, Resistor_THT:R_Axial_DIN0207_L6.3mm_D2.5mm_P7.62mm_Horizontal, F.Cu at (164.0, 37.8)
- added R25: 100, Resistor_THT:R_Axial_DIN0207_L6.3mm_D2.5mm_P7.62mm_Horizontal, F.Cu at (164.0, 41.9)
- added R26: 100, Resistor_THT:R_Axial_DIN0207_L6.3mm_D2.5mm_P7.62mm_Horizontal, F.Cu at (164.0, 45.9)
- added R27: 100, Resistor_THT:R_Axial_DIN0207_L6.3mm_D2.5mm_P7.62mm_Horizontal, F.Cu at (164.0, 50.0)
- added R3: 2.2, Resistor_THT:R_Axial_DIN0207_L6.3mm_D2.5mm_P7.62mm_Horizontal, F.Cu at (142.4, 33.8)
- added R4: 2.2, Resistor_THT:R_Axial_DIN0207_L6.3mm_D2.5mm_P7.62mm_Horizontal, F.Cu at (142.4, 37.8)
- added R5: 2.2, Resistor_THT:R_Axial_DIN0207_L6.3mm_D2.5mm_P7.62mm_Horizontal, F.Cu at (142.4, 41.9)
- added R6: 100, Resistor_THT:R_Axial_DIN0207_L6.3mm_D2.5mm_P7.62mm_Horizontal, F.Cu at (142.4, 45.9)
- added R7: 100, Resistor_THT:R_Axial_DIN0207_L6.3mm_D2.5mm_P7.62mm_Horizontal, F.Cu at (142.4, 50.0)
- added R8: 100, Resistor_THT:R_Axial_DIN0207_L6.3mm_D2.5mm_P7.62mm_Horizontal, F.Cu at (142.4, 54.0)
- added R9: 100, Resistor_THT:R_Axial_DIN0207_L6.3mm_D2.5mm_P7.62mm_Horizontal, F.Cu at (142.4, 58.1)
- moved U1 126.9 mm to (211.5, 145.1)
- moved A1 100.2 mm to (97.0, 127.5)
- moved Q15 37.5 mm to (95.0, 93.0)
- moved D9 9.57 mm to (59.4, 119.5)
Connections:
- A1 pad 15: Net-(A1-D0/RX) -> unconnected-(A1-D0/RX-Pad15)
- U1 pad 1: Net-(A1-D0/RX) -> unconnected-(U1-RO-Pad1)

Commit message: pcd one
Parts:
- moved R21 242.8 mm to (45.0, 237.3)
- moved R23 242.8 mm to (45.0, 245.4)
- moved R22 242.8 mm to (45.0, 241.3)
- moved C3 213.8 mm to (33.2, 241.5)
- moved R19 207.8 mm to (26.2, 222.5)
- moved R25 202.0 mm to (96.0, 232.1)
- moved R24 202.0 mm to (96.0, 228.0)
- moved R26 202.0 mm to (96.0, 236.1)
- moved R27 202.0 mm to (96.0, 240.2)
- moved R20 200.8 mm to (44.7, 231.0)
- moved J12 187.3 mm to (83.0, 239.5)
- moved J11 186.8 mm to (82.0, 228.2)
- moved R15 175.1 mm to (32.3, 168.5)
- moved J10 170.6 mm to (66.5, 240.6)
- moved J9 170.6 mm to (66.5, 230.5)
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Routing:
- net +5V: track 0.00 -> 17.3 mm
- net GND: track 0.00 -> 16.6 mm

Commit message: pcd built
Parts:
- D1: footprint Diode_THT:D_DO-35_SOD27_P10.16mm_Horizontal -> Diode_THT:D_DO-35_SOD27_P7.62mm_Horizontal
- moved R23 228.7 mm to (105.3, 24.8), turned to -90 degrees
- moved C3 227.9 mm to (138.6, 39.4), turned to -90 degrees
- moved R19 226.2 mm to (152.8, 35.0)
- moved R22 221.0 mm to (83.4, 23.7), turned to -90 degrees
- moved Q15 218.9 mm to (124.0, 33.0), turned to 90 degrees
- moved R21 214.6 mm to (59.3, 23.2), turned to -90 degrees
- moved R20 208.4 mm to (39.2, 22.7), turned to -90 degrees
- moved J10 199.2 mm to (59.9, 41.5), turned to -90 degrees
- moved J12 198.2 mm to (105.7, 42.6), turned to -90 degrees
- moved J9 190.8 mm to (39.8, 41.6), turned to -90 degrees
- moved Q9 190.6 mm to (40.2, 59.2), turned to 90 degrees
- moved Q12 187.7 mm to (105.7, 59.6), turned to 90 degrees
- moved J11 187.3 mm to (82.5, 40.9), turned to -90 degrees
- moved Q10 187.0 mm to (59.6, 59.3), turned to 90 degrees
- moved Q11 184.3 mm to (82.4, 59.9), turned to 90 degrees
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Routing:
- net +5V: track 17.3 -> 612.5 mm
- net Net-(A1-D6): track 0.00 -> 94.6 mm
- net Net-(D9-K): track 0.00 -> 73.1 mm
- net Net-(A1-D3): track 0.00 -> 71.3 mm
- net Net-(D3-K): track 0.00 -> 69.8 mm
- net Net-(D6-K): track 0.00 -> 69.0 mm
- net Net-(A1-D11): track 0.00 -> 51.2 mm
- net Net-(A1-D5): track 0.00 -> 50.6 mm
- net Net-(A1-D9): track 0.00 -> 39.9 mm
- net Net-(Q15-B): track 0.00 -> 35.4 mm
- net Net-(Q14-B): track 0.00 -> 34.6 mm
- net Net-(Q13-B): track 0.00 -> 28.4 mm
- net Net-(D1-K): track 0.00 -> 24.2 mm
- net Net-(D2-K): track 0.00 -> 23.3 mm
- net Net-(Q8-B): track 0.00 -> 22.6 mm
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
Commit message: updated pcb
Parts:
- U1: footprint Package_SO:SOIC-8_3.9x4.9mm_P1.27mm -> rosekicad:MAX485_Module
- moved R6 61.2 mm to (75.8, 156.8)
- moved D1 58.2 mm to (78.5, 167.2), turned to 0 degrees
- moved R7 56.1 mm to (89.8, 156.5)
- moved D2 55.0 mm to (93.5, 167.5), turned to 0 degrees
- moved D3 54.4 mm to (108.2, 167.5), turned to 0 degrees
- moved Q1 52.8 mm to (70.8, 153.2)
- moved R8 51.6 mm to (104.8, 157.0)
- moved R9 49.9 mm to (118.6, 156.5)
- moved Q2 48.3 mm to (84.6, 153.3)
- moved J1 48.2 mm to (70.8, 139.0)
- moved C4 46.9 mm to (303.5, 97.5), turned to 180 degrees
- moved C1 46.4 mm to (139.2, 125.5)
- moved R1 46.4 mm to (148.9, 125.5)
- moved Q3 44.5 mm to (99.1, 153.8)
- moved R2 43.5 mm to (70.8, 124.2)
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Connections:
- D2 pad 1: Net-(D2-K) -> Net-(D1-A)
- D2 pad 2: Net-(D1-K) -> Net-(D2-A)
- D3 pad 1: Net-(D3-K) -> Net-(D2-A)
- D3 pad 2: Net-(D2-K) -> Net-(D3-A)
- D5 pad 1: Net-(D5-K) -> Net-(D4-A)
- D5 pad 2: Net-(D4-K) -> Net-(D5-A)
- D6 pad 1: Net-(D6-K) -> Net-(D5-A)
- D6 pad 2: Net-(D5-K) -> Net-(D6-A)
- D8 pad 1: Net-(D8-K) -> Net-(D7-A)
- D8 pad 2: Net-(D7-K) -> Net-(D8-A)
- D9 pad 1: Net-(D9-K) -> Net-(D8-A)
- D9 pad 2: Net-(D8-K) -> Net-(D9-A)
- Q13 pad 1: Net-(D3-K) -> Net-(D3-A)
- Q14 pad 1: Net-(D6-K) -> Net-(D6-A)
- Q15 pad 1: Net-(D9-K) -> Net-(D9-A)
- R15 pad 2: Net-(D4-A) -> Net-(D4-K)
- R16 pad 2: Net-(D4-K) -> Net-(D4-A)
- R17 pad 2: Net-(D5-K) -> Net-(D5-A)
- R18 pad 2: Net-(D6-K) -> Net-(D6-A)
- R24 pad 2: Net-(D7-A) -> Net-(D7-K)
- R25 pad 2: Net-(D7-K) -> Net-(D7-A)
- R26 pad 2: Net-(D8-K) -> Net-(D8-A)
- R27 pad 2: Net-(D9-K) -> Net-(D9-A)
- R6 pad 2: Net-(D1-A) -> Net-(D1-K)
- R7 pad 2: Net-(D1-K) -> Net-(D1-A)
- R8 pad 2: Net-(D2-K) -> Net-(D2-A)
- R9 pad 2: Net-(D3-K) -> Net-(D3-A)
Routing:
- net +5V: track 612.5 -> 485.1 mm
- net Net-(A1-D1/TX): track 0.00 -> 85.2 mm
- net GND: track 17.6 -> 92.4 mm
- net Net-(D9-K): track 73.1 -> 0.00 mm
- net Net-(D3-K): track 69.8 -> 0.00 mm
- net Net-(D6-K): track 69.0 -> 0.00 mm
- net Net-(A1-+5V): track 0.00 -> 54.3 mm
- net Net-(D3-A): track 0.00 -> 50.0 mm
- net Net-(D6-A): track 0.00 -> 48.8 mm
- net Net-(A1-D6): track 94.6 -> 49.7 mm
- net Net-(D9-A): track 0.00 -> 43.2 mm
- net Net-(D2-K): track 23.3 -> 0.00 mm
- net Net-(D8-K): track 21.7 -> 0.00 mm
- net Net-(D5-K): track 21.4 -> 0.00 mm
- net Net-(D1-K): track 24.2 -> 4.98 mm
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
Commit message: Added four layers
Parts:
- moved C5 200.9 mm to (105.0, 146.0), turned to 180 degrees
- moved C4 170.2 mm to (135.2, 123.0), turned to 90 degrees
- moved J16 159.3 mm to (121.3, 124.0), turned to 0 degrees
- moved J15 126.3 mm to (165.0, 111.0)
- moved U1 115.7 mm to (142.0, 114.0), turned to -90 degrees
- moved J13 84.5 mm to (134.0, 97.0), turned to -90 degrees
- moved J14 66.2 mm to (119.0, 97.0), turned to -90 degrees
- moved A1 60.5 mm to (163.0, 80.0), turned to 180 degrees
- moved R1 56.8 mm to (96.0, 105.0)
- moved R10 51.3 mm to (97.5, 65.0)
- moved R19 48.9 mm to (97.5, 17.5)
- moved C1 45.2 mm to (94.0, 127.1)
- moved Q13 44.7 mm to (82.3, 128.3)
- moved Q14 44.7 mm to (83.1, 79.2)
- moved C2 44.6 mm to (94.3, 77.8)
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Routing:
- net +5V: track 485.1 -> 4.21 mm
- net GND: track 92.4 -> 0.00 mm
- net Net-(A1-D9): track 20.9 -> 102.9 mm
- net Net-(A1-D6): track 49.7 -> 128.8 mm
- net Net-(A1-D5): track 50.6 -> 112.3 mm
- net Net-(A1-+5V): track 54.3 -> 0.00 mm
- net Net-(A1-D3): track 71.3 -> 114.5 mm
- net Net-(A1-D1/TX): track 85.2 -> 111.4 mm
- net Net-(J15-Pin_2): track 12.9 -> 31.1 mm
- net Net-(J15-Pin_3): track 11.9 -> 24.6 mm
- net Net-(Q13-B): track 22.1 -> 34.6 mm
- net Net-(A1-D11): track 58.0 -> 63.8 mm
- net Net-(Q14-B): track 19.6 -> 25.2 mm
- net Net-(D3-A): track 50.0 -> 47.1 mm
- net Net-(Q15-B): track 20.3 -> 22.5 mm
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- added copper zone on In2.Cu, net +5V
- added copper zone on In1.Cu, net GND
Other:
- copper layers 2 -> 4

Commit message: mounting holes
Parts:
- added H1: MountingHole, MountingHole:MountingHole_4.5mm_Pad, F.Cu at (276.9, 38.1)
- added H2: MountingHole, MountingHole:MountingHole_4.5mm_Pad, F.Cu at (99.1, 38.1)
- added H3: MountingHole, MountingHole:MountingHole_4.5mm_Pad, F.Cu at (99.1, 190.5)
- added H4: MountingHole, MountingHole:MountingHole_4.5mm_Pad, F.Cu at (276.9, 190.5)
- moved J11 83.8 mm to (140.3, 62.4)
- moved J10 83.7 mm to (125.5, 62.4)
- moved J9 83.7 mm to (110.8, 62.4)
- moved C3 83.6 mm to (175.6, 53.9)
- moved J12 83.6 mm to (154.3, 62.4)
- moved Q12 83.6 mm to (154.6, 76.7)
- moved Q15 83.6 mm to (163.8, 55.2)
- moved R19 83.6 mm to (176.9, 43.8)
- moved R23 83.6 mm to (154.3, 46.4)
- moved R25 83.6 mm to (130.1, 80.2)
- moved R26 83.6 mm to (145.6, 80.2)
- moved R27 83.6 mm to (158.8, 79.7)
- moved A1 83.6 mm to (242.4, 106.3)
- moved C1 83.6 mm to (173.4, 153.3)
- moved C2 83.6 mm to (173.7, 104.0)
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Connections:
- A1 pad 5: Net-(A1-+5V) -> +5V
- C4 pad 1: Net-(A1-+5V) -> +5V
- U1 pad 1: unconnected-(U1-RO-Pad1) -> Net-(A1-D1/TX)
- U1 pad 4: Net-(A1-D1/TX) -> unconnected-(U1-DI-Pad4)
- U1 pad 8: Net-(A1-+5V) -> +5V
Other:
- board outline added: 203.2 x 177.8 mm

Commit message: finalized pcb main
Parts:
- moved J15 48.9 mm to (202.2, 162.0), turned to 0 degrees
- moved R1 42.7 mm to (148.6, 164.5)
- moved J13 37.8 mm to (179.1, 139.1)
- moved J14 36.9 mm to (165.1, 139.1)
- moved R10 36.1 mm to (148.6, 113.7)
- moved R19 34.2 mm to (148.6, 62.9)
- moved R18 33.2 mm to (133.3, 149.3)
- moved Q8 33.0 mm to (128.3, 146.7)
- moved H1 32.9 mm to (252.7, 60.4)
- moved D6 32.7 mm to (123.2, 159.5)
- moved Q12 32.6 mm to (128.3, 96.0)
- moved R9 32.4 mm to (132.1, 197.6)
- moved R23 32.3 mm to (128.3, 65.5)
- moved J8 32.1 mm to (128.3, 131.5)
- moved R14 32.0 mm to (128.3, 116.5)
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Connections:
- A1 pad 15: unconnected-(A1-D0/RX-Pad15) -> Net-(A1-D0/RX)
- A1 pad 16: Net-(A1-D1/TX) -> unconnected-(A1-D1/TX-Pad16)
- U1 pad 1: Net-(A1-D1/TX) -> Net-(A1-D0/RX)
Routing:
- net Net-(A1-D1/TX): track 111.4 -> 0.00 mm
- net Net-(A1-D0/RX): track 0.00 -> 85.0 mm
- net Net-(J15-Pin_3): track 24.6 -> 51.6 mm
- net Net-(A1-D6): track 128.8 -> 147.8 mm
- net Net-(J15-Pin_2): track 31.1 -> 49.9 mm
- net Net-(A1-D3): track 114.5 -> 95.8 mm
- net Net-(Q13-B): track 34.6 -> 19.4 mm
- net Net-(A1-D9): track 102.9 -> 112.4 mm
- net Net-(A1-D11): track 63.8 -> 72.5 mm
- net Net-(D9-A): track 43.2 -> 49.6 mm
- net Net-(Q14-B): track 25.2 -> 19.4 mm
- net Net-(A1-D5): track 112.3 -> 107.4 mm
- net Net-(D7-K): track 7.86 -> 3.43 mm
- net +5V: track 4.21 -> 0.00 mm
- net Net-(D8-A): track 11.0 -> 7.62 mm
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Other:
- board size 203.2 x 177.8 mm -> 190.5 x 165.1 mm
- board text added: "Anna Tretiakova Levitating Rose Project 205 Spring 2026 https://github.com/Shapitsa/Rose-Electronics-Senior-Design"
